File: kicad_files/hope-s.kicad_pcb (KiCad board)
At the start: 2 copper layers, 344.7 x 123.1 mm, 256 parts, among them J1 EXTRA_PINS, J2 TYPE-C-31-M-12, Q1 2N7002, Q2 2N7002, Q3 2N7002, Q4 2N7002, Q5 AO3401A, Q6 2N7002, SW1 K2-1187SQ-A4SW-06, SW10 MX Switch, SW100 MX Switch, SW101 MX Switch, SW102 MX Switch, SW103 MX Switch, SW104 MX Switch, SW11 MX Switch, SW12 MX Switch, SW13 MX Switch, SW14 MX Switch, SW15 MX Switch, SW16 MX Switch, SW17 MX Switch, SW18 MX Switch, SW19 MX Switch, SW2 MX Switch, SW20 MX Switch, SW21 MX Switch, SW22 MX Switch, SW23 MX Switch, SW24 MX Switch, SW25 MX Switch, SW26 MX Switch, SW27 MX Switch, SW28 MX Switch, SW29 MX Switch, SW3 MX Switch, SW30 MX Switch, SW31 MX Switch, SW32 MX Switch, SW33 MX Switch, SW34 MX Switch, SW35 MX Switch, SW36 MX Switch, SW37 MX Switch, SW38 MX Switch, SW39 MX Switch, SW4 MX Switch, SW40 MX Switch, SW41 MX Switch, SW42 MX Switch, SW43 MX Switch, SW44 MX Switch, SW45 MX Switch, SW46 MX Switch, SW47 MX Switch, SW48 MX Switch, SW49 MX Switch, SW5 MX Switch, SW50 MX Switch, SW51 MX Switch, SW52 MX Switch, SW53 MX Switch, SW54 MX Switch, SW55 MX Switch, SW56 MX Switch, SW57 MX Switch, SW58 MX Switch, SW59 MX Switch, SW6 MX Switch, SW60 MX Switch, SW61 MX Switch, SW62 MX Switch, SW63 MX Switch, SW64 MX Switch, SW65 MX Switch, SW66 MX Switch, SW67 MX Switch, SW68 MX Switch, SW69 MX Switch, SW7 MX Switch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

Commit message: Remove components lib
Parts:
- removed D36: 1N4148W, acheron_Components:D_SOD-123
- moved R4 303.2 mm to (269.4, 157.6)
- moved D2 20.8 mm to (316.4, 98.2)
- moved U3 20.8 mm to (313.0, 97.7)
- moved R14 20.8 mm to (319.6, 98.9)
- moved D37 19.0 mm to (346.9, 131.1)
- moved D38 17.7 mm to (327.8, 131.1)
- moved D12 7.62 mm to (165.9, 88.3)
- moved D3 6.73 mm to (351.6, 88.3)
- moved D11 4.91 mm to (194.5, 88.3)
- moved D15 4.76 mm to (108.7, 88.3)
- moved D9 4.76 mm to (232.6, 88.3)
- moved D10 4.76 mm to (213.5, 88.3)
- moved D8 4.76 mm to (251.6, 88.3)
- moved D13 2.66 mm to (146.8, 88.3)
- moved D4 2.66 mm to (337.3, 88.3)
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Routing:
- net R2: track 286.0 -> 308.6 mm
- net Net-(D9-A): track 0.00 -> 20.9 mm
- net Net-(D8-A): track 0.00 -> 20.9 mm
- net Net-(D10-A): track 0.00 -> 20.9 mm
- net Net-(D3-A): track 0.00 -> 15.1 mm
- net Net-(D36-A): track 0.00 -> 14.8 mm
- net Net-(D51-A): track 0.00 -> 12.7 mm
- net Net-(D39-A): track 0.00 -> 10.5 mm
- net Net-(D38-A): track 0.00 -> 10.5 mm
- net Net-(D7-A): track 0.00 -> 10.5 mm
- net Net-(D6-A): track 0.00 -> 10.5 mm
- net Net-(D53-A): track 0.00 -> 10.5 mm
- net Net-(D24-A): track 0.00 -> 10.5 mm
- net Net-(D47-A): track 0.00 -> 10.5 mm
- net Net-(D46-A): track 0.00 -> 10.5 mm
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